Commit message: kdl test and rrbot urdf update

File: rover_ws/src/hal_description/urdf/rrbot.xacro (robot description, xacro)
@@ -12,7 +12,7 @@
   <xacro:property name="axel_offset" value="0.05" /> <!-- Space btw top of beam and the each joint -->
   <!-- Import all Gazebo-customization elements, including Gazebo colors -->
-  <xacro:include filename="$(find rrbot_description)/urdf/rrbot.gazebo" />
+  <xacro:include filename="$(find hal_description)/urdf/rrbot.gazebo" />
   <!-- Import Rviz colors -->
-  <xacro:include filename="$(find rrbot_description)/urdf/materials.xacro" />
+  <xacro:include filename="$(find hal_description)/urdf/materials.xacro" />
   <!-- Used for fixing robot to Gazebo 'base_link' -->
   <link name="world"/>
@@ -107,76 +107,76 @@
     </inertial>
   </link>
-  <joint name="hokuyo_joint" type="fixed">
-    <axis xyz="0 1 0" />
-    <origin xyz="0 0 ${height3 - axel_offset/2}" rpy="0 0 0"/>
-    <parent link="link3"/>
-    <child link="hokuyo_link"/>
-  </joint>
+<!--  <joint name="hokuyo_joint" type="fixed">-->
+<!--    <axis xyz="0 1 0" />-->
+<!--    <origin xyz="0 0 ${height3 - axel_offset/2}" rpy="0 0 0"/>-->
+<!--    <parent link="link3"/>-->
+<!--    <child link="hokuyo_link"/>-->
+<!--  </joint>-->
   <!-- Hokuyo Laser -->
-  <link name="hokuyo_link">
-    <collision>
-      <origin xyz="0 0 0" rpy="0 0 0"/>
-      <geometry>
-	<box size="0.1 0.1 0.1"/>
-      </geometry>
-    </collision>
-    <visual>
-      <origin xyz="0 0 0" rpy="0 0 0"/>
-      <geometry>
-        <mesh filename="package://rrbot_description/meshes/hokuyo.dae"/>
-      </geometry>
-    </visual>
-    <inertial>
-      <mass value="1e-5" />
-      <origin xyz="0 0 0" rpy="0 0 0"/>
-      <inertia ixx="1e-6" ixy="0" ixz="0" iyy="1e-6" iyz="0" izz="1e-6" />
-    </inertial>
-  </link>
-  <joint name="camera_joint" type="fixed">
-    <axis xyz="0 1 0" />
-    <origin xyz="${camera_link} 0 ${height3 - axel_offset*2}" rpy="0 0 0"/>
-    <parent link="link3"/>
-    <child link="camera_link"/>
-  </joint>
+<!--  <link name="hokuyo_link">-->
+<!--    <collision>-->
+<!--      <origin xyz="0 0 0" rpy="0 0 0"/>-->
+<!--      <geometry>-->
+<!--	<box size="0.1 0.1 0.1"/>-->
+<!--      </geometry>-->
+<!--    </collision>-->
+<!--    <visual>-->
+<!--      <origin xyz="0 0 0" rpy="0 0 0"/>-->
+<!--      <geometry>-->
+<!--        <mesh filename="package://hal_description/meshes/hokuyo.dae"/>-->
+<!--      </geometry>-->
+<!--    </visual>-->
+<!--    <inertial>-->
+<!--      <mass value="1e-5" />-->
+<!--      <origin xyz="0 0 0" rpy="0 0 0"/>-->
+<!--      <inertia ixx="1e-6" ixy="0" ixz="0" iyy="1e-6" iyz="0" izz="1e-6" />-->
+<!--    </inertial>-->
+<!--  </link>-->
+<!--  <joint name="camera_joint" type="fixed">-->
+<!--    <axis xyz="0 1 0" />-->
+<!--    <origin xyz="${camera_link} 0 ${height3 - axel_offset*2}" rpy="0 0 0"/>-->
+<!--    <parent link="link3"/>-->
+<!--    <child link="camera_link"/>-->
+<!--  </joint>-->
   <!-- Camera -->
-  <link name="camera_link">
-    <collision>
-      <origin xyz="0 0 0" rpy="0 0 0"/>
-      <geometry>
-	<box size="${camera_link} ${camera_link} ${camera_link}"/>
-      </geometry>
-    </collision>
-    <visual>
-      <origin xyz="0 0 0" rpy="0 0 0"/>
-      <geometry>
-	<box size="${camera_link} ${camera_link} ${camera_link}"/>
-      </geometry>
-      <material name="red"/>
-    </visual>
-    <inertial>
-      <mass value="1e-5" />
-      <origin xyz="0 0 0" rpy="0 0 0"/>
-      <inertia ixx="1e-6" ixy="0" ixz="0" iyy="1e-6" iyz="0" izz="1e-6" />
-    </inertial>
-  </link>
-  <transmission name="tran1">
-    <type>transmission_interface/SimpleTransmission</type>
-    <joint name="joint1">
-      <hardwareInterface>EffortJointInterface</hardwareInterface>
-    </joint>
-    <actuator name="motor1">
-      <hardwareInterface>EffortJointInterface</hardwareInterface>
-      <mechanicalReduction>1</mechanicalReduction>
-    </actuator>
-  </transmission>
-  <transmission name="tran2">
-    <type>transmission_interface/SimpleTransmission</type>
-    <joint name="joint2">
-      <hardwareInterface>EffortJointInterface</hardwareInterface>
-    </joint>
-    <actuator name="motor2">
-      <hardwareInterface>EffortJointInterface</hardwareInterface>
-      <mechanicalReduction>1</mechanicalReduction>
-    </actuator>
-  </transmission>
+<!--  <link name="camera_link">-->
+<!--    <collision>-->
+<!--      <origin xyz="0 0 0" rpy="0 0 0"/>-->
+<!--      <geometry>-->
+<!--	<box size="${camera_link} ${camera_link} ${camera_link}"/>-->
+<!--      </geometry>-->
+<!--    </collision>-->
+<!--    <visual>-->
+<!--      <origin xyz="0 0 0" rpy="0 0 0"/>-->
+<!--      <geometry>-->
+<!--	<box size="${camera_link} ${camera_link} ${camera_link}"/>-->
+<!--      </geometry>-->
+<!--      <material name="red"/>-->
+<!--    </visual>-->
+<!--    <inertial>-->
+<!--      <mass value="1e-5" />-->
+<!--      <origin xyz="0 0 0" rpy="0 0 0"/>-->
+<!--      <inertia ixx="1e-6" ixy="0" ixz="0" iyy="1e-6" iyz="0" izz="1e-6" />-->
+<!--    </inertial>-->
+<!--  </link>-->
+<!--  <transmission name="tran1">-->
+<!--    <type>transmission_interface/SimpleTransmission</type>-->
+<!--    <joint name="joint1">-->
+<!--      <hardwareInterface>EffortJointInterface</hardwareInterface>-->
+<!--    </joint>-->
+<!--    <actuator name="motor1">-->
+<!--      <hardwareInterface>EffortJointInterface</hardwareInterface>-->
+<!--      <mechanicalReduction>1</mechanicalReduction>-->
+<!--    </actuator>-->
+<!--  </transmission>-->
+<!--  <transmission name="tran2">-->
+<!--    <type>transmission_interface/SimpleTransmission</type>-->
+<!--    <joint name="joint2">-->
+<!--      <hardwareInterface>EffortJointInterface</hardwareInterface>-->
+<!--    </joint>-->
+<!--    <actuator name="motor2">-->
+<!--      <hardwareInterface>EffortJointInterface</hardwareInterface>-->
+<!--      <mechanicalReduction>1</mechanicalReduction>-->
+<!--    </actuator>-->
+<!--  </transmission>-->
 </robot>
