Commit message: Add dummy link to arm URDF

File: rover_ws/src/hal_description/urdf/rover_arm.xacro (robot description, xacro)
@@ -220,5 +220,5 @@
       <origin xyz="0 ${-(d6-dyn)/2} 0" rpy="0 0 0"/>
       <geometry>
-	<box size="${width} ${d6-dyn} ${width}"/>
+				<box size="${width} ${d6-dyn} ${width}"/>
       </geometry>
     </collision>
@@ -226,5 +226,5 @@
       <origin xyz="0 ${-(d6-dyn)/2} 0" rpy="0 0 0"/>
       <geometry>
-	<box size="${width} ${d6-dyn} ${width}"/>
+				<box size="${width} ${d6-dyn} ${width}"/>
       </geometry>
       <material name="white"/>
@@ -239,3 +239,25 @@
     </inertial>
   </link>
+  <joint name="joint7" type="fixed">
+		<parent link="link7"/>
+		<child link="end"/>
+		<origin xyz="0 ${-(d6-dyn)} 0" rpy="0 0 0"/>
+	</joint>
+	<!-- Dummy Link to force KDL chain point to tip of claw -->
+	<link name="end">
+		<visual>
+			<geometry>
+				<box size="0 0 0"/>
+			</geometry>
+		</visual>
+		<inertial>
+			<origin xyz="0 0 0" rpy="0 0 0"/>
+			<mass value="0"/>
+			<inertia
+				ixx="0" ixy="0" ixz="0"
+				iyy="0" iyz="0"
+				izz="0"
+			/>
+		</inertial>
+	</link>
 </robot>

Commit message: "Added Approximate Joint Limits"

File: rover_ws/src/hal_description/urdf/rover_arm.xacro (robot description, xacro)
@@ -17,4 +17,6 @@
   <xacro:property name="dyn" value="0" /> <!-- Dynamixel length -->
   <xacro:property name="axel_offset" value="0.05" /> <!-- Space btw top of beam and the each joint -->
+  <xacro:property name="Torque" value = "40" />
+  <xacro:property name="vel" value = "10" />
   <!-- Import all Gazebo-customization elements, including Gazebo colors -->
   <xacro:include filename="$(find hal_description)/urdf/hal.gazebo" />
@@ -84,5 +86,5 @@
   </link>
   <!-- Turret up/down -->
-  <joint name="joint2" type="continuous">
+  <joint name="joint2" type="revolute">
     <parent link="link2"/>
     <child link="link3"/>
@@ -90,4 +92,5 @@
     <axis xyz="1 0 0"/>
     <dynamics damping="0.7"/>
+    <limit effort="${Torque}" velocity="${vel}" lower="${-PI/2}" upper="${PI/2}" />
   </joint>
   <!-- Tube 1  -->
@@ -115,5 +118,5 @@
     </inertial>
   </link>
-  <joint name="joint3" type="continuous">
+  <joint name="joint3" type="revolute">
     <parent link="link3"/>
     <child link="link4"/>
@@ -121,4 +124,5 @@
     <axis xyz="1 0 0"/>
     <dynamics damping="0.7"/>
+    <limit effort="${Torque}" velocity="${vel}" lower="${-PI}" upper="${PI}" />
   </joint>
 <!-- Offset Length -->
