Commit message: 537 project: progress on 537.xacro of rover base

File: rover_ws/src/hal_description/urdf/537.urdf (robot description, URDF)
Before this commit: robot rrbot, 2 links, 1 joints
Links:
- removed link world
- added link base_link
- added link box1; visual box size=0.25 0.5 0.25
- added link fork1; visual box size=0.1 0.75 0.1
- added link fork2; visual box size=0.1 0.75 0.1
- added link rffork1; visual box size=0.1 0.75 0.1
Joints:
- added joint topplate_to_box: type fixed, parent base1, child box1, origin xyz=0.4318 0 0.40005
- added joint topplate_to_frontfork1: type fixed, parent base1, child fork1, origin xyz=-0.4318 0 0.40005
- added joint topplate_to_frontfork2: type fixed, parent base1, child fork2, origin xyz=-0.4318 0 0.40005
- added joint topplate_to_rightfrontfork1: type fixed, parent base1, child rffork1, origin xyz=0 0 0.40005
- joint fixed: child link1 -> base1; parent world -> base_link

File: rover_ws/src/hal_description/urdf/rover_complete_537.xacro (robot description, xacro)
@@ -45,5 +45,6 @@
       <origin xyz="0 0 ${flattop_offground + (1/2)*flattopheight}" rpy="0 0 0"/>
       <geometry>
-	<box size="${flattoplength} ${flattopwidth} ${flattopheight}"/>
+	  <box size="${flattoplength} ${flattopwidth} ${flattopheight}"/>
+	  <box size="1.0 1.0 1.0"/>
       </geometry>
       <material name="white"/>

Commit message: 537 urdf with collision

File: rover_ws/src/hal_description/urdf/537.urdf (robot description, URDF)
Before this commit: robot 537_base, 6 links, 5 joints
Links:
- removed link rffork1
- link base1: geometry collision box size=0.8636 0.6096 0.0254; visual box size=0.8636 0.6096 0.0254
- link box1: geometry collision box size=0.25 0.5 0.25; visual box size=0.25 0.5 0.25
- link fork1: geometry collision box size=0.1 0.75 0.1; visual box size=0.1 0.75 0.1
- link fork2: geometry collision box size=0.1 0.75 0.1; visual box size=0.1 0.75 0.1
Joints:
- removed joint topplate_to_rightfrontfork1

File: rover_ws/src/hal_description/urdf/537.xacro (robot description, xacro)
@@ -36,4 +36,11 @@
       <material name="white"/>
     </visual>
+    <collision>
+      <origin xyz="0 0 ${flattop_offground + (1/2)*flattopheight}" rpy="0 0 0"/>
+        <geometry>
+	       <box size="${flattoplength} ${flattopwidth} ${flattopheight}"/>
+        </geometry>
+      <material name="white"/>
+    </collision>
   </link>
    <joint name="topplate_to_box" type="fixed">
@@ -51,4 +58,11 @@
       <material name="white"/>
     </visual>
+    <collision>
+      <origin xyz="${-0.5*boxwidth} 0 ${(1/2)*boxheight}" rpy="0 0 0"/>
+        <geometry>
+         <box size="${boxwidth} ${boxlength} ${boxheight}"/>
+        </geometry>
+      <material name="white"/>
+    </collision>
   </link>
 <!-- Joint from top plate to back fork -->
@@ -67,4 +81,11 @@
       <material name="white"/>
     </visual>
+    <collision>
+      <origin xyz="${-bforkwidth/2} ${0.5*bforklength} ${-0.771*bforklength/2}" rpy="${-45*PI/180} 0 0"/>
+        <geometry>
+         <box size="${bforkwidth} ${bforklength} ${bforkheight}"/>
+        </geometry>
+      <material name="white"/>
+    </collision>
   </link>
 <!-- Joint from top plate to back fork -->
@@ -83,13 +104,21 @@
       <material name="white"/>
     </visual>
+    <collision>
+      <origin xyz="${-bforkwidth/2} ${-0.5*bforklength} ${-0.771*bforklength/2}" rpy="${45*PI/180} 0 0"/>
+        <geometry>
+         <box size="${bforkwidth} ${bforklength} ${bforkheight}"/>
+        </geometry>
+      <material name="white"/>
+    </collision>
   </link>
 <!-- Joint from top plate to right front fork -->
-   <joint name="topplate_to_rightfrontfork1" type="fixed">
+<!--    <joint name="topplate_to_rightfrontfork1" type="fixed">
     <parent link="base1"/>
     <child link="rffork1"/>
     <origin xyz="0 0 ${flattop_offground + flattopheight}"/>
   </joint>
+ -->
 <!-- Back Fork Link -->
-  <link name="rffork1">
+<!--   <link name="rffork1">
     <visual>
       <origin xyz="${-bforkwidth/2} ${-0.5*bforklength} ${-0.771*bforklength/2}" rpy="${45*PI/180} 0 0"/>
@@ -99,5 +128,5 @@
       <material name="white"/>
     </visual>
-  </link>
+  </link>   -->
   <!-- Turret-->
 <!--   <joint name="joint1" type="continuous">
